File: opensbc.kicad_sch (KiCad schematic)
At the start: 5 parts, among them U1 MIMX8MN5DVPIZDA, U2 B3221PM3BDGUI, U3 B3221PM3BDGUI, U4 EMMC32G-TS0A-01002, U5 PCA9450BHNY

Commit message: Revert "Schematic progress"
This reverts commit 0ab4f18268ae0280199bb3a3efdd6a38bd66ed97.
Connections:
- removed net CA0_A: U1.R1 (DRAM_AC08), U2.H2 (CA0_A), U3.H2 (CA0_A)
- removed net CA0_B: U1.AA3 (DRAM_AC28), U2.R2 (CA0_B), U3.R2 (CA0_B)
- removed net CA1_A: U1.R2 (DRAM_AC09), U2.J2 (CA1_A), U3.J2 (CA1_A)
- removed net CA1_B: U1.V4 (DRAM_AC29), U2.P2 (CA1_B), U3.P2 (CA1_B)
- removed net CA2_A: U1.M2 (DRAM_AC10), U2.H9 (CA2_A), U3.H9 (CA2_A)
- removed net CA2_B: U1.W1 (DRAM_AC30), U2.R9 (CA2_B), U3.R9 (CA2_B)
- removed net CA3_A: U1.L2 (DRAM_AC11), U2.H10 (CA3_A), U3.H10 (CA3_A)
- removed net CA3_B: U1.Y3 (DRAM_AC31), U2.R10 (CA3_B), U3.R10 (CA3_B)
- removed net CA4_A: U1.L1 (DRAM_AC12), U2.H11 (CA4_A), U3.H11 (CA4_A)
- removed net CA4_B: U1.R5 (DRAM_AC32), U2.R11 (CA4_B), U3.R11 (CA4_B)
- removed net CA5_A: U1.M1 (DRAM_AC13), U2.J11 (CA5_A), U3.J11 (CA5_A)
- removed net CA5_B: U1.U2 (DRAM_AC33), U2.P11 (CA5_B), U3.P11 (CA5_B)
- removed net CKE0_A: U1.P1 (DRAM_AC00), U2.J4 (CKE0_A), U3.J4 (CKE0_A)
- removed net CKE0_B: U1.T1 (DRAM_AC20), U2.P4 (CKE0_B), U3.P4 (CKE0_B)
- removed net CKE1_A: U1.N1 (DRAM_AC01), U2.J5 (CKE1_A), U3.J5 (CKE1_A)
- removed net CKE1_B: U1.T2 (DRAM_AC21), U2.P5 (CKE1_B), U3.P5 (CKE1_B)
- net CK_c_A: no longer names the net of U1.G4 (DRAM_AC05)
- removed net CK_c_B: U1.AA2 (DRAM_AC25), U2.P9 (CK_c_B), U3.P9 (CK_c_B)
- removed net CK_t_A: U1.G5 (DRAM_AC04), U2.J8 (CK_t_A), U3.J8 (CK_t_A)
- removed net CK_t_B: U1.Y2 (DRAM_AC24), U2.P8 (CK_t_B), U3.P8 (CK_t_B)
- removed net CS0_A: U1.N2 (DRAM_AC02), U2.H4 (CS0_A), U3.H4 (CS0_A)
- net CS0_B: no longer names the net of U1.R4 (DRAM_AC23)
- removed net CS1_A: U1.P2 (DRAM_AC03), U2.H3 (CS1_A), U3.H3 (CS1_A)
- removed net DRAM_DATA0: U1.B3 (DRAM_DQ00), U2.B2 (DQ0_A), U3.B2 (DQ0_A)
- removed net DRAM_DATA1: U1.A2 (DRAM_DQ01), U2.C2 (DQ1_A), U3.C2 (DQ1_A)
- removed net DRAM_DATA10: U1.J1 (DRAM_DQ10), U2.E11 (DQ10_A), U3.E11 (DQ10_A)
- removed net DRAM_DATA11: U1.J2 (DRAM_DQ11), U2.F11 (DQ11_A), U3.F11 (DQ11_A)
- removed net DRAM_DATA12: U1.K1 (DRAM_DQ12), U2.F9 (DQ12_A), U3.F9 (DQ12_A)
- removed net DRAM_DATA13: U1.K2 (DRAM_DQ13), U2.E9 (DQ13_A), U3.E9 (DQ13_A)
- removed net DRAM_DATA14: U1.F2 (DRAM_DQ14), U2.C9 (DQ14_A), U3.C9 (DQ14_A)
- removed net DRAM_DATA15: U1.E1 (DRAM_DQ15), U2.B9 (DQ15_A), U3.B9 (DQ15_A)
- removed net DRAM_DATA2: U1.A3 (DRAM_DQ02), U2.E2 (DQ2_A), U3.E2 (DQ2_A)
- removed net DRAM_DATA3: U1.B4 (DRAM_DQ03), U2.F2 (DQ3_A), U3.F2 (DQ3_A)
- removed net DRAM_DATA4: U1.E2 (DRAM_DQ04), U2.F4 (DQ4_A), U3.F4 (DQ4_A)
- removed net DRAM_DATA5: U1.D1 (DRAM_DQ05), U2.E4 (DQ5_A), U3.E4 (DQ5_A)
- removed net DRAM_DATA6: U1.C1 (DRAM_DQ06), U2.C4 (DQ6_A), U3.C4 (DQ6_A)
- removed net DRAM_DATA7: U1.D2 (DRAM_DQ07), U2.B4 (DQ7_A), U3.B4 (DQ7_A)
- removed net DRAM_DATA8: U1.G1 (DRAM_DQ08), U2.B11 (DQ8_A), U3.B11 (DQ8_A)
- removed net DRAM_DATA9: U1.H1 (DRAM_DQ09), U2.C11 (DQ9_A), U3.C11 (DQ9_A)
- removed net DRAM_DMI0: U1.B2 (DRAM_DM0), U2.C3 (DMI0_A), U3.C3 (DMI0_A)
- removed net DRAM_DMI1: U1.H2 (DRAM_DM1), U2.C10 (DMI1_A), U3.C10 (DMI1_A)
- removed net DRAM_DQS0_N: U1.C2 (DRAM_DQS0_N), U2.E3 (DQS0_c_A), U3.E3 (DQS0_c_A)
- removed net DRAM_DQS0_P: U1.B1 (DRAM_DQS0_P), U2.D3 (DQS0_t_A), U3.D3 (DQS0_t_A)
- removed net DRAM_DQS1_N: U1.F1 (DRAM_DQS1_N), U2.E10 (DQS1_c_A), U3.E10 (DQS1_c_A)
- removed net DRAM_DQS1_P: U1.G2 (DRAM_DQS1_P), U2.D10 (DQS1_t_A), U3.D10 (DQS1_t_A)
- net DRAM_NRST: no longer names the net of U1.N4 (DRAM_RESET_N)
- net DRAM_NRST: no longer U2.T11 (NRST)
- net DRAM_VREF: no longer names the net of U1.L4 (DRAM_VREF)
- net DRAM_ZQ: no longer names the net of U1.U1 (DRAM_ZN)
- no-connect marks 10 -> 0
Other:
- moved on the sheet: U1D, U1E, U2A, U2B, U3A, U3B, U4

Commit message: Schematic progress
Connections:
- net DRAM_DATA1: now reaches U1.A2 (DRAM_DQ01)
- net DRAM_DATA1: now also U2.C2 (DQ1_A), U3.C2 (DQ1_A)
- net DRAM_DATA2: now reaches U1.A3 (DRAM_DQ02)
- net DRAM_DATA2: now also U2.E2 (DQ2_A), U3.E2 (DQ2_A)
- net CK_c_B: now reaches U1.AA2 (DRAM_AC25)
- net CK_c_B: now also U2.P9 (CK_c_B), U3.P9 (CK_c_B)
- net CA0_B: now reaches U1.AA3 (DRAM_AC28)
- net CA0_B: now also U2.R2 (CA0_B), U3.R2 (CA0_B)
- net DRAM_DQS0_P: now reaches U1.B1 (DRAM_DQS0_P)
- net DRAM_DQS0_P: now also U2.D3 (DQS0_t_A), U3.D3 (DQS0_t_A)
- net DRAM_DMI0: now reaches U1.B2 (DRAM_DM0)
- net DRAM_DMI0: now also U2.C3 (DMI0_A), U3.C3 (DMI0_A)
- net DRAM_DATA0: now reaches U1.B3 (DRAM_DQ00)
- net DRAM_DATA0: now also U2.B2 (DQ0_A), U3.B2 (DQ0_A)
- net DRAM_DATA3: now reaches U1.B4 (DRAM_DQ03)
- net DRAM_DATA3: now also U2.F2 (DQ3_A), U3.F2 (DQ3_A)
- net DRAM_DATA6: now reaches U1.C1 (DRAM_DQ06)
- net DRAM_DATA6: now also U2.C4 (DQ6_A), U3.C4 (DQ6_A)
- net DRAM_DQS0_N: now reaches U1.C2 (DRAM_DQS0_N)
- net DRAM_DQS0_N: now also U2.E3 (DQS0_c_A), U3.E3 (DQS0_c_A)
- net DRAM_DATA5: now reaches U1.D1 (DRAM_DQ05)
- net DRAM_DATA5: now also U2.E4 (DQ5_A), U3.E4 (DQ5_A)
- net DRAM_DATA7: now reaches U1.D2 (DRAM_DQ07)
- net DRAM_DATA7: now also U2.B4 (DQ7_A), U3.B4 (DQ7_A)
- net DRAM_DATA15: now reaches U1.E1 (DRAM_DQ15)
- net DRAM_DATA15: now also U2.B9 (DQ15_A), U3.B9 (DQ15_A)
- net DRAM_DATA4: now reaches U1.E2 (DRAM_DQ04)
- net DRAM_DATA4: now also U2.F4 (DQ4_A), U3.F4 (DQ4_A)
- net DRAM_DQS1_N: now reaches U1.F1 (DRAM_DQS1_N)
- net DRAM_DQS1_N: now also U2.E10 (DQS1_c_A), U3.E10 (DQS1_c_A)
- net DRAM_DATA14: now reaches U1.F2 (DRAM_DQ14)
- net DRAM_DATA14: now also U2.C9 (DQ14_A), U3.C9 (DQ14_A)
- net DRAM_DATA8: now reaches U1.G1 (DRAM_DQ08)
- net DRAM_DATA8: now also U2.B11 (DQ8_A), U3.B11 (DQ8_A)
- net DRAM_DQS1_P: now reaches U1.G2 (DRAM_DQS1_P)
- net DRAM_DQS1_P: now also U2.D10 (DQS1_t_A), U3.D10 (DQS1_t_A)
- net CK_c_A: now reaches U1.G4 (DRAM_AC05)
- net CK_t_A: now reaches U1.G5 (DRAM_AC04)
- net CK_t_A: now also U2.J8 (CK_t_A), U3.J8 (CK_t_A)
- net DRAM_DATA9: now reaches U1.H1 (DRAM_DQ09)
- net DRAM_DATA9: now also U2.C11 (DQ9_A), U3.C11 (DQ9_A)
- net DRAM_DMI1: now reaches U1.H2 (DRAM_DM1)
- net DRAM_DMI1: now also U2.C10 (DMI1_A), U3.C10 (DMI1_A)
- net DRAM_DATA10: now reaches U1.J1 (DRAM_DQ10)
- net DRAM_DATA10: now also U2.E11 (DQ10_A), U3.E11 (DQ10_A)
- net DRAM_DATA11: now reaches U1.J2 (DRAM_DQ11)
- net DRAM_DATA11: now also U2.F11 (DQ11_A), U3.F11 (DQ11_A)
- net DRAM_DATA12: now reaches U1.K1 (DRAM_DQ12)
- net DRAM_DATA12: now also U2.F9 (DQ12_A), U3.F9 (DQ12_A)
- net DRAM_DATA13: now reaches U1.K2 (DRAM_DQ13)
- net DRAM_DATA13: now also U2.E9 (DQ13_A), U3.E9 (DQ13_A)
- net CA4_A: now reaches U1.L1 (DRAM_AC12)
- net CA4_A: now also U2.H11 (CA4_A), U3.H11 (CA4_A)
- net CA3_A: now reaches U1.L2 (DRAM_AC11)
- net CA3_A: now also U2.H10 (CA3_A), U3.H10 (CA3_A)
- net DRAM_VREF: now reaches U1.L4 (DRAM_VREF)
- net CA5_A: now reaches U1.M1 (DRAM_AC13)
- net CA5_A: now also U2.J11 (CA5_A), U3.J11 (CA5_A)
- net CA2_A: now reaches U1.M2 (DRAM_AC10)
- net CA2_A: now also U2.H9 (CA2_A), U3.H9 (CA2_A)
- net CKE1_A: now reaches U1.N1 (DRAM_AC01)
- net CKE1_A: now also U2.J5 (CKE1_A), U3.J5 (CKE1_A)
- net CS0_A: now reaches U1.N2 (DRAM_AC02)
- net CS0_A: now also U2.H4 (CS0_A), U3.H4 (CS0_A)
- net DRAM_NRST: now reaches U1.N4 (DRAM_RESET_N)
- net DRAM_NRST: now also U2.T11 (NRST)
- net CKE0_A: now reaches U1.P1 (DRAM_AC00)
- net CKE0_A: now also U2.J4 (CKE0_A), U3.J4 (CKE0_A)
- net CS1_A: now reaches U1.P2 (DRAM_AC03)
- net CS1_A: now also U2.H3 (CS1_A), U3.H3 (CS1_A)
- net CA0_A: now reaches U1.R1 (DRAM_AC08)
- net CA0_A: now also U2.H2 (CA0_A), U3.H2 (CA0_A)
- net CA1_A: now reaches U1.R2 (DRAM_AC09)
- net CA1_A: now also U2.J2 (CA1_A), U3.J2 (CA1_A)
- net CS0_B: now reaches U1.R4 (DRAM_AC23)
- net CA4_B: now reaches U1.R5 (DRAM_AC32)
- net CA4_B: now also U2.R11 (CA4_B), U3.R11 (CA4_B)
- net CKE0_B: now reaches U1.T1 (DRAM_AC20)
- net CKE0_B: now also U2.P4 (CKE0_B), U3.P4 (CKE0_B)
- net CKE1_B: now reaches U1.T2 (DRAM_AC21)
- net CKE1_B: now also U2.P5 (CKE1_B), U3.P5 (CKE1_B)
- net DRAM_ZQ: now reaches U1.U1 (DRAM_ZN)
- net CA5_B: now reaches U1.U2 (DRAM_AC33)
- net CA5_B: now also U2.P11 (CA5_B), U3.P11 (CA5_B)
- net CA1_B: now reaches U1.V4 (DRAM_AC29)
- net CA1_B: now also U2.P2 (CA1_B), U3.P2 (CA1_B)
- net CA2_B: now reaches U1.W1 (DRAM_AC30)
- net CA2_B: now also U2.R9 (CA2_B), U3.R9 (CA2_B)
- net CK_t_B: now reaches U1.Y2 (DRAM_AC24)
- net CK_t_B: now also U2.P8 (CK_t_B), U3.P8 (CK_t_B)
- net CA3_B: now reaches U1.Y3 (DRAM_AC31)
- net CA3_B: now also U2.R10 (CA3_B), U3.R10 (CA3_B)
- no-connect marks 0 -> 10
Other:
- moved on the sheet: U1D, U1E, U2A, U2B, U3A, U3B, U4
