File: opensbc.kicad_pcb (KiCad board)
At the start: 8 copper layers, 5 parts, among them U1 MIMX8MN5DVPIZDA, U2 B3221PM3BDGUI, U3 B3221PM3BDGUI, U4 EMMC32G-TS0A-01002, U5 PCA9450BHNY

Commit message: Schematic progress
Connections:
- U1 pad A2: unconnected-(U1C-DRAM_DQ01-PadA2) -> /DRAM_DATA1
- U1 pad A3: unconnected-(U1C-DRAM_DQ02-PadA3) -> /DRAM_DATA2
- U1 pad B1: unconnected-(U1C-DRAM_DQS0_P-PadB1) -> /DRAM_DQS0_P
- U1 pad B2: unconnected-(U1C-DRAM_DM0-PadB2) -> /DRAM_DMI0
- U1 pad B3: unconnected-(U1C-DRAM_DQ00-PadB3) -> /DRAM_DATA0
- U1 pad B4: unconnected-(U1C-DRAM_DQ03-PadB4) -> /DRAM_DATA3
- U1 pad C1: unconnected-(U1C-DRAM_DQ06-PadC1) -> /DRAM_DATA6
- U1 pad C2: unconnected-(U1C-DRAM_DQS0_N-PadC2) -> /DRAM_DQS0_N
- U1 pad D1: unconnected-(U1C-DRAM_DQ05-PadD1) -> /DRAM_DATA5
- U1 pad D2: unconnected-(U1C-DRAM_DQ07-PadD2) -> /DRAM_DATA7
- U1 pad E1: unconnected-(U1C-DRAM_DQ15-PadE1) -> /DRAM_DATA15
- U1 pad E2: unconnected-(U1C-DRAM_DQ04-PadE2) -> /DRAM_DATA4
- U1 pad F1: unconnected-(U1C-DRAM_DQS1_N-PadF1) -> /DRAM_DQS1_N
- U1 pad F2: unconnected-(U1C-DRAM_DQ14-PadF2) -> /DRAM_DATA14
- U1 pad G1: unconnected-(U1C-DRAM_DQ08-PadG1) -> /DRAM_DATA8
- U1 pad G2: unconnected-(U1C-DRAM_DQS1_P-PadG2) -> /DRAM_DQS1_P
- U1 pad H1: unconnected-(U1C-DRAM_DQ09-PadH1) -> /DRAM_DATA9
- U1 pad H2: unconnected-(U1C-DRAM_DM1-PadH2) -> /DRAM_DMI1
- U1 pad J1: unconnected-(U1C-DRAM_DQ10-PadJ1) -> /DRAM_DATA10
- U1 pad J2: unconnected-(U1C-DRAM_DQ11-PadJ2) -> /DRAM_DATA11
- U1 pad K1: unconnected-(U1C-DRAM_DQ12-PadK1) -> /DRAM_DATA12
- U1 pad K2: unconnected-(U1C-DRAM_DQ13-PadK2) -> /DRAM_DATA13
- U2 pad B11: unconnected-(U2B-DQ8_A-PadB11) -> /DRAM_DATA8
- U2 pad B2: unconnected-(U2B-DQ0_A-PadB2) -> /DRAM_DATA0
- U2 pad B4: unconnected-(U2B-DQ7_A-PadB4) -> /DRAM_DATA7
- U2 pad B9: unconnected-(U2B-DQ15_A-PadB9) -> /DRAM_DATA15
- U2 pad C10: unconnected-(U2B-DMI1_A-PadC10) -> /DRAM_DMI1
- U2 pad C11: unconnected-(U2B-DQ9_A-PadC11) -> /DRAM_DATA9
- U2 pad C2: unconnected-(U2B-DQ1_A-PadC2) -> /DRAM_DATA1
- U2 pad C3: unconnected-(U2B-DMI0_A-PadC3) -> /DRAM_DMI0
- U2 pad C4: unconnected-(U2B-DQ6_A-PadC4) -> /DRAM_DATA6
- U2 pad C9: unconnected-(U2B-DQ14_A-PadC9) -> /DRAM_DATA14
- U2 pad D10: unconnected-(U2B-DQS1_t_A-PadD10) -> /DRAM_DQS1_P
- U2 pad D3: unconnected-(U2B-DQS0_t_A-PadD3) -> /DRAM_DQS0_P
- U2 pad E10: unconnected-(U2B-DQS1_c_A-PadE10) -> /DRAM_DQS1_N
- U2 pad E11: unconnected-(U2B-DQ10_A-PadE11) -> /DRAM_DATA10
- U2 pad E2: unconnected-(U2B-DQ2_A-PadE2) -> /DRAM_DATA2
- U2 pad E3: unconnected-(U2B-DQS0_c_A-PadE3) -> /DRAM_DQS0_N
- U2 pad E4: unconnected-(U2B-DQ5_A-PadE4) -> /DRAM_DATA5
- U2 pad E9: unconnected-(U2B-DQ13_A-PadE9) -> /DRAM_DATA13
- U2 pad F11: unconnected-(U2B-DQ11_A-PadF11) -> /DRAM_DATA11
- U2 pad F2: unconnected-(U2B-DQ3_A-PadF2) -> /DRAM_DATA3
- U2 pad F4: unconnected-(U2B-DQ4_A-PadF4) -> /DRAM_DATA4
- U2 pad F9: unconnected-(U2B-DQ12_A-PadF9) -> /DRAM_DATA12
- U3 pad B11: unconnected-(U3B-DQ8_A-PadB11) -> /DRAM_DATA8
- U3 pad B2: unconnected-(U3B-DQ0_A-PadB2) -> /DRAM_DATA0
- U3 pad B4: unconnected-(U3B-DQ7_A-PadB4) -> /DRAM_DATA7
- U3 pad B9: unconnected-(U3B-DQ15_A-PadB9) -> /DRAM_DATA15
- U3 pad C10: unconnected-(U3B-DMI1_A-PadC10) -> /DRAM_DMI1
- U3 pad C11: unconnected-(U3B-DQ9_A-PadC11) -> /DRAM_DATA9
- U3 pad C2: unconnected-(U3B-DQ1_A-PadC2) -> /DRAM_DATA1
- U3 pad C3: unconnected-(U3B-DMI0_A-PadC3) -> /DRAM_DMI0
- U3 pad C4: unconnected-(U3B-DQ6_A-PadC4) -> /DRAM_DATA6
- U3 pad C9: unconnected-(U3B-DQ14_A-PadC9) -> /DRAM_DATA14
- U3 pad D10: unconnected-(U3B-DQS1_t_A-PadD10) -> /DRAM_DQS1_P
- U3 pad D3: unconnected-(U3B-DQS0_t_A-PadD3) -> /DRAM_DQS0_P
- U3 pad E10: unconnected-(U3B-DQS1_c_A-PadE10) -> /DRAM_DQS1_N
- U3 pad E11: unconnected-(U3B-DQ10_A-PadE11) -> /DRAM_DATA10
- U3 pad E2: unconnected-(U3B-DQ2_A-PadE2) -> /DRAM_DATA2
- U3 pad E3: unconnected-(U3B-DQS0_c_A-PadE3) -> /DRAM_DQS0_N
- U3 pad E4: unconnected-(U3B-DQ5_A-PadE4) -> /DRAM_DATA5
- U3 pad E9: unconnected-(U3B-DQ13_A-PadE9) -> /DRAM_DATA13
- U3 pad F11: unconnected-(U3B-DQ11_A-PadF11) -> /DRAM_DATA11
- U3 pad F2: unconnected-(U3B-DQ3_A-PadF2) -> /DRAM_DATA3
- U3 pad F4: unconnected-(U3B-DQ4_A-PadF4) -> /DRAM_DATA4
- U3 pad F9: unconnected-(U3B-DQ12_A-PadF9) -> /DRAM_DATA12

Commit message: Revert "Schematic progress"
This reverts commit 0ab4f18268ae0280199bb3a3efdd6a38bd66ed97.
Connections:
- U1 pad A2: /DRAM_DATA1 -> unconnected-(U1C-DRAM_DQ01-PadA2)
- U1 pad A3: /DRAM_DATA2 -> unconnected-(U1C-DRAM_DQ02-PadA3)
- U1 pad B1: /DRAM_DQS0_P -> unconnected-(U1C-DRAM_DQS0_P-PadB1)
- U1 pad B2: /DRAM_DMI0 -> unconnected-(U1C-DRAM_DM0-PadB2)
- U1 pad B3: /DRAM_DATA0 -> unconnected-(U1C-DRAM_DQ00-PadB3)
- U1 pad B4: /DRAM_DATA3 -> unconnected-(U1C-DRAM_DQ03-PadB4)
- U1 pad C1: /DRAM_DATA6 -> unconnected-(U1C-DRAM_DQ06-PadC1)
- U1 pad C2: /DRAM_DQS0_N -> unconnected-(U1C-DRAM_DQS0_N-PadC2)
- U1 pad D1: /DRAM_DATA5 -> unconnected-(U1C-DRAM_DQ05-PadD1)
- U1 pad D2: /DRAM_DATA7 -> unconnected-(U1C-DRAM_DQ07-PadD2)
- U1 pad E1: /DRAM_DATA15 -> unconnected-(U1C-DRAM_DQ15-PadE1)
- U1 pad E2: /DRAM_DATA4 -> unconnected-(U1C-DRAM_DQ04-PadE2)
- U1 pad F1: /DRAM_DQS1_N -> unconnected-(U1C-DRAM_DQS1_N-PadF1)
- U1 pad F2: /DRAM_DATA14 -> unconnected-(U1C-DRAM_DQ14-PadF2)
- U1 pad G1: /DRAM_DATA8 -> unconnected-(U1C-DRAM_DQ08-PadG1)
- U1 pad G2: /DRAM_DQS1_P -> unconnected-(U1C-DRAM_DQS1_P-PadG2)
- U1 pad H1: /DRAM_DATA9 -> unconnected-(U1C-DRAM_DQ09-PadH1)
- U1 pad H2: /DRAM_DMI1 -> unconnected-(U1C-DRAM_DM1-PadH2)
- U1 pad J1: /DRAM_DATA10 -> unconnected-(U1C-DRAM_DQ10-PadJ1)
- U1 pad J2: /DRAM_DATA11 -> unconnected-(U1C-DRAM_DQ11-PadJ2)
- U1 pad K1: /DRAM_DATA12 -> unconnected-(U1C-DRAM_DQ12-PadK1)
- U1 pad K2: /DRAM_DATA13 -> unconnected-(U1C-DRAM_DQ13-PadK2)
- U2 pad B11: /DRAM_DATA8 -> unconnected-(U2B-DQ8_A-PadB11)
- U2 pad B2: /DRAM_DATA0 -> unconnected-(U2B-DQ0_A-PadB2)
- U2 pad B4: /DRAM_DATA7 -> unconnected-(U2B-DQ7_A-PadB4)
- U2 pad B9: /DRAM_DATA15 -> unconnected-(U2B-DQ15_A-PadB9)
- U2 pad C10: /DRAM_DMI1 -> unconnected-(U2B-DMI1_A-PadC10)
- U2 pad C11: /DRAM_DATA9 -> unconnected-(U2B-DQ9_A-PadC11)
- U2 pad C2: /DRAM_DATA1 -> unconnected-(U2B-DQ1_A-PadC2)
- U2 pad C3: /DRAM_DMI0 -> unconnected-(U2B-DMI0_A-PadC3)
- U2 pad C4: /DRAM_DATA6 -> unconnected-(U2B-DQ6_A-PadC4)
- U2 pad C9: /DRAM_DATA14 -> unconnected-(U2B-DQ14_A-PadC9)
- U2 pad D10: /DRAM_DQS1_P -> unconnected-(U2B-DQS1_t_A-PadD10)
- U2 pad D3: /DRAM_DQS0_P -> unconnected-(U2B-DQS0_t_A-PadD3)
- U2 pad E10: /DRAM_DQS1_N -> unconnected-(U2B-DQS1_c_A-PadE10)
- U2 pad E11: /DRAM_DATA10 -> unconnected-(U2B-DQ10_A-PadE11)
- U2 pad E2: /DRAM_DATA2 -> unconnected-(U2B-DQ2_A-PadE2)
- U2 pad E3: /DRAM_DQS0_N -> unconnected-(U2B-DQS0_c_A-PadE3)
- U2 pad E4: /DRAM_DATA5 -> unconnected-(U2B-DQ5_A-PadE4)
- U2 pad E9: /DRAM_DATA13 -> unconnected-(U2B-DQ13_A-PadE9)
- U2 pad F11: /DRAM_DATA11 -> unconnected-(U2B-DQ11_A-PadF11)
- U2 pad F2: /DRAM_DATA3 -> unconnected-(U2B-DQ3_A-PadF2)
- U2 pad F4: /DRAM_DATA4 -> unconnected-(U2B-DQ4_A-PadF4)
- U2 pad F9: /DRAM_DATA12 -> unconnected-(U2B-DQ12_A-PadF9)
- U3 pad B11: /DRAM_DATA8 -> unconnected-(U3B-DQ8_A-PadB11)
- U3 pad B2: /DRAM_DATA0 -> unconnected-(U3B-DQ0_A-PadB2)
- U3 pad B4: /DRAM_DATA7 -> unconnected-(U3B-DQ7_A-PadB4)
- U3 pad B9: /DRAM_DATA15 -> unconnected-(U3B-DQ15_A-PadB9)
- U3 pad C10: /DRAM_DMI1 -> unconnected-(U3B-DMI1_A-PadC10)
- U3 pad C11: /DRAM_DATA9 -> unconnected-(U3B-DQ9_A-PadC11)
- U3 pad C2: /DRAM_DATA1 -> unconnected-(U3B-DQ1_A-PadC2)
- U3 pad C3: /DRAM_DMI0 -> unconnected-(U3B-DMI0_A-PadC3)
- U3 pad C4: /DRAM_DATA6 -> unconnected-(U3B-DQ6_A-PadC4)
- U3 pad C9: /DRAM_DATA14 -> unconnected-(U3B-DQ14_A-PadC9)
- U3 pad D10: /DRAM_DQS1_P -> unconnected-(U3B-DQS1_t_A-PadD10)
- U3 pad D3: /DRAM_DQS0_P -> unconnected-(U3B-DQS0_t_A-PadD3)
- U3 pad E10: /DRAM_DQS1_N -> unconnected-(U3B-DQS1_c_A-PadE10)
- U3 pad E11: /DRAM_DATA10 -> unconnected-(U3B-DQ10_A-PadE11)
- U3 pad E2: /DRAM_DATA2 -> unconnected-(U3B-DQ2_A-PadE2)
- U3 pad E3: /DRAM_DQS0_N -> unconnected-(U3B-DQS0_c_A-PadE3)
- U3 pad E4: /DRAM_DATA5 -> unconnected-(U3B-DQ5_A-PadE4)
- U3 pad E9: /DRAM_DATA13 -> unconnected-(U3B-DQ13_A-PadE9)
- U3 pad F11: /DRAM_DATA11 -> unconnected-(U3B-DQ11_A-PadF11)
- U3 pad F2: /DRAM_DATA3 -> unconnected-(U3B-DQ3_A-PadF2)
- U3 pad F4: /DRAM_DATA4 -> unconnected-(U3B-DQ4_A-PadF4)
- U3 pad F9: /DRAM_DATA12 -> unconnected-(U3B-DQ12_A-PadF9)
